Commit message: Update: 자크로 오류

File: f1tenth_gym_ros/launch/ego_racecar.xacro (robot description, xacro)
@@ -40,5 +40,5 @@
     </visual>
   </link>
-  <joint name="$base_to_back_left_wheel" type="fixed">
+  <joint name="base_to_back_left_wheel" type="fixed">
     <parent link="${car_name}/base_link"/>
     <child link="${car_name}/back_left_wheel"/>
