Commit message: 라이프사이클 매니저 수정 및 프레임 이름 변경 (완)

File: simulator/urdf/ego_racecar.xacro (robot description, xacro)
@@ -11,5 +11,4 @@
   <xacro:property name="laser_height" value="0.05" />
   <xacro:property name="laser_radius" value="0.026" />
-  <xacro:property name="car_name" value="ego_racecar" />
   <material name="black">
     <color rgba="0.2 0.2 0.2 1."/>
@@ -18,5 +17,5 @@
     <color rgba="0.3 0.57 1. 1."/>
   </material>
-  <link name="${car_name}/base_link">
+  <link name="base_link">
     <visual>
       <origin xyz="${wheelbase/2} 0 ${ground_offset+height/2}"/>
@@ -28,9 +27,9 @@
   </link>
   <joint name="base_to_laser_model" type="fixed">
-    <parent link="${car_name}/base_link"/>
-    <child link="${car_name}/laser_model"/>
+    <parent link="base_link"/>
+    <child link="laser_model"/>
     <origin xyz="${laser_distance_from_base_link} 0 ${ground_offset+height+(laser_height/2)}"/>
   </joint>
-  <link name="${car_name}/laser_model">
+  <link name="laser_model">
     <visual>
       <geometry>
@@ -41,9 +40,9 @@
   </link>
   <joint name="base_to_back_left_wheel" type="fixed">
-    <parent link="${car_name}/base_link"/>
-    <child link="${car_name}/back_left_wheel"/>
+    <parent link="base_link"/>
+    <child link="back_left_wheel"/>
     <origin xyz="0 ${(wheel_length+width)/2} ${wheel_radius}"/>
   </joint>
-  <link name="${car_name}/back_left_wheel">
+  <link name="back_left_wheel">
     <visual>
       <geometry>
@@ -55,9 +54,9 @@
   </link>
   <joint name="base_to_back_right_wheel" type="fixed">
-    <parent link="${car_name}/base_link"/>
-    <child link="${car_name}/back_right_wheel"/>
+    <parent link="base_link"/>
+    <child link="back_right_wheel"/>
     <origin xyz="0 ${-(wheel_length+width)/2} ${wheel_radius}"/>
   </joint>
-  <link name="${car_name}/back_right_wheel">
+  <link name="back_right_wheel">
     <visual>
       <geometry>
@@ -69,14 +68,14 @@
   </link>
   <joint name="base_to_front_left_hinge" type="fixed">
-    <parent link="${car_name}/base_link"/>
-    <child link="${car_name}/front_left_hinge"/>
+    <parent link="base_link"/>
+    <child link="front_left_hinge"/>
     <origin xyz="${wheelbase} ${(wheel_length+width)/2} ${wheel_radius}"/>
   </joint>
-  <link name="${car_name}/front_left_hinge"/>
+  <link name="front_left_hinge"/>
   <joint name="front_left_hinge_to_wheel" type="continuous">
-    <parent link="${car_name}/front_left_hinge"/>
-    <child link="${car_name}/front_left_wheel"/>
+    <parent link="front_left_hinge"/>
+    <child link="front_left_wheel"/>
   </joint>
-  <link name="${car_name}/front_left_wheel">
+  <link name="front_left_wheel">
     <visual>
       <geometry>
@@ -88,14 +87,14 @@
   </link>
   <joint name="base_to_front_right_hinge" type="fixed">
-    <parent link="${car_name}/base_link"/>
-    <child link="${car_name}/front_right_hinge"/>
+    <parent link="base_link"/>
+    <child link="front_right_hinge"/>
     <origin xyz="${wheelbase} ${-(wheel_length+width)/2} ${wheel_radius}"/>
   </joint>
-  <link name="${car_name}/front_right_hinge"/>
+  <link name="front_right_hinge"/>
   <joint name="front_right_hinge_to_wheel" type="continuous">
-    <parent link="${car_name}/front_right_hinge"/>
-    <child link="${car_name}/front_right_wheel"/>
+    <parent link="front_right_hinge"/>
+    <child link="front_right_wheel"/>
   </joint>
-  <link name="${car_name}/front_right_wheel">
+  <link name="front_right_wheel">
     <visual>
       <geometry>
